Commit message: modified

File: src/description/robot_core.xacro (robot description, xacro)
@@ -40,9 +40,9 @@
     <link name="link_1">
         <visual>
-            <!-- <origin xyz="0 0 ${link_1_length/2}" rpy="0 0 0"/> -->
-            <origin xyz="0 0 0" rpy="0 0 ${-pi/2}"/>
+            <origin xyz="0 0 ${link_1_length/2}" rpy="0 0 0"/>
+            <!-- <origin xyz="0 0 0" rpy="0 0 ${-pi/2}"/> -->
             <geometry>
-                <!-- <cylinder length="${link_1_length}" radius="${link_1_radius}" /> -->
-                 <mesh filename="package://arm_bot/meshes/puma_link1.stl" scale="0.0254 0.0254 0.0254"/>
+                <cylinder length="${link_1_length}" radius="${link_1_radius}" />
+                 <!-- <mesh filename="package://3_link_arm/meshes/puma_link1.stl" scale="0.0254 0.0254 0.0254"/> -->
             </geometry>
             <material name="purple" />
@@ -52,5 +52,5 @@
             <geometry>
                 <cylinder length="${link_1_length}" radius="${link_1_radius}" />
-                 <!-- <mesh filename="package://arm_bot/meshes/puma_link1.stl" scale="0.0254 0.0254 0.0254"/> -->
+                 <!-- <mesh filename="package://3_link_arm/meshes/puma_link1.stl" scale="0.0254 0.0254 0.0254"/> -->
             </geometry>
         </collision>
@@ -67,5 +67,5 @@
         <child link="shoulder"/>
         <axis xyz="0 0 1"/>
-        <limit lower="${-8*pi/9}" upper="${8*pi/9}" velocity="2" effort="1000"/>
+        <limit lower="${-10*pi}" upper="${10*pi}" velocity="2" effort="1000"/>
         <dynamics damping="0" friction="0"/>
     </joint>
@@ -73,9 +73,9 @@
     <link name="shoulder">
         <visual>
-            <!-- <origin xyz="0 ${shoulder_length/2 - shoulder_radius} 0" rpy="${pi/2} 0 0"/> -->
-            <origin xyz="0 -0.09677 0" rpy="${pi/2} 0 ${pi}"/>
+            <origin xyz="0 ${shoulder_length/2 - shoulder_radius} 0" rpy="${pi/2} 0 0"/>
+            <!-- <origin xyz="0 -0.09677 0" rpy="${pi/2} 0 ${pi}"/> -->
             <geometry>
-                <!-- <cylinder length="${shoulder_length}" radius="${shoulder_radius}" /> -->
-                 <mesh filename="package://arm_bot/meshes/puma_link2.stl" scale="0.0254 0.0254 0.0254"/>
+                <cylinder length="${shoulder_length}" radius="${shoulder_radius}" />
+                 <!-- <mesh filename="package://3_link_arm/meshes/puma_link2.stl" scale="0.0254 0.0254 0.0254"/> -->
             </geometry>
             <material name="blue" />
@@ -98,5 +98,5 @@
         <child link="link_2"/>
         <axis xyz="0 0 1"/>
-        <limit lower="${-5*pi/4}" upper="${pi/4}" velocity="2" effort="1000"/>
+        <limit lower="${-10*pi}" upper="${10*pi}" velocity="2" effort="1000"/>
         <dynamics damping="0" friction="0"/>
     </joint>
@@ -105,9 +105,9 @@
     <link name="link_2">
         <visual>
-            <!-- <origin xyz="${link_2_length/2} 0 0" rpy="0 ${pi/2} 0"/> -->
-            <origin xyz="0 0 0" rpy="0 0 0"/>
+            <origin xyz="${link_2_length/2} 0 0" rpy="0 ${pi/2} 0"/>
+            <!-- <origin xyz="0 0 0" rpy="0 0 0"/> -->
             <geometry>
-                <!-- <cylinder length="${link_2_length}" radius="${link_2_radius}" /> -->
-                 <mesh filename="package://arm_bot/meshes/puma_link3.stl" scale="0.0254 0.0254 0.0254"/>
+                <cylinder length="${link_2_length}" radius="${link_2_radius}" />
+                 <!-- <mesh filename="package://3_link_arm/meshes/puma_link3.stl" scale="0.0254 0.0254 0.0254"/> -->
             </geometry>
             <material name="orange" />
@@ -130,5 +130,5 @@
         <child link="link_3"/>
         <axis xyz="0 0 1"/>
-        <limit lower="${-pi/4}" upper="${5*pi/4}" velocity="2" effort="1000"/>
+        <limit lower="${-10*pi}" upper="${10*pi}" velocity="2" effort="1000"/>
         <dynamics damping="0" friction="0"/>
     </joint>
@@ -137,9 +137,9 @@
     <link name="link_3">
         <visual>
-            <!-- <origin xyz="0 -${link_3_length/2} 0" rpy="${-pi/2} 0 0"/> -->
-            <origin xyz="0 ${0.094/2} 0" rpy="0 0 ${-pi/2}"/>
+            <origin xyz="0 -${link_3_length/2} 0" rpy="${-pi/2} 0 0"/>
+            <!-- <origin xyz="0 ${0.094/2} 0" rpy="0 0 ${-pi/2}"/> -->
             <geometry>
-                <!-- <cylinder length="${link_3_length}" radius="${link_3_radius}" /> -->
-                 <mesh filename="package://arm_bot/meshes/puma_link4.stl" scale="0.0254 0.0254 0.0254"/>
+                <cylinder length="${link_3_length}" radius="${link_3_radius}" />
+                 <!-- <mesh filename="package://3_link_arm/meshes/puma_link4.stl" scale="0.0254 0.0254 0.0254"/> -->
             </geometry>
             <material name="yellow" />

File: src/description/ros2_control.xacro (robot description, xacro)
@@ -7,5 +7,5 @@
             </hardware>
             <joint name="joint_1">
-                <command_interface name="effort"/>
+                <command_interface name="velocity"/>
                 <state_interface name="velocity"/>
                 <state_interface name="position"/>
@@ -13,5 +13,5 @@
             </joint>
             <joint name="joint_2">
-                <command_interface name="effort"/>
+                <command_interface name="velocity"/>
                 <state_interface name="velocity"/>
                 <state_interface name="position"/>
@@ -19,5 +19,5 @@
             </joint>
             <joint name="joint_3">
-                <command_interface name="effort"/>
+                <command_interface name="velocity"/>
                 <state_interface name="velocity"/>
                 <state_interface name="position"/>
@@ -28,6 +28,6 @@
     <gazebo>
         <plugin name="gazebo_ros2_control" filename="libgazebo_ros2_control.so">
-            <parameters>$(find arm_bot)/config/my_controllers.yaml</parameters>
-            <parameters>$(find arm_bot)/config/gaz_ros2_ctl_use_sim.yaml</parameters>
+            <parameters>$(find 3_link_arm)/config/my_controllers.yaml</parameters>
+            <parameters>$(find 3_link_arm)/config/gaz_ros2_ctl_use_sim.yaml</parameters>
         </plugin>
     </gazebo>

Commit message: comments deleted

File: src/description/robot_core.xacro (robot description, xacro)
@@ -41,8 +41,6 @@
         <visual>
             <origin xyz="0 0 ${link_1_length/2}" rpy="0 0 0"/>
-            <!-- <origin xyz="0 0 0" rpy="0 0 ${-pi/2}"/> -->
             <geometry>
                 <cylinder length="${link_1_length}" radius="${link_1_radius}" />
-                 <!-- <mesh filename="package://3_link_arm/meshes/puma_link1.stl" scale="0.0254 0.0254 0.0254"/> -->
             </geometry>
             <material name="purple" />
@@ -52,5 +50,4 @@
             <geometry>
                 <cylinder length="${link_1_length}" radius="${link_1_radius}" />
-                 <!-- <mesh filename="package://3_link_arm/meshes/puma_link1.stl" scale="0.0254 0.0254 0.0254"/> -->
             </geometry>
         </collision>
@@ -74,8 +71,6 @@
         <visual>
             <origin xyz="0 ${shoulder_length/2 - shoulder_radius} 0" rpy="${pi/2} 0 0"/>
-            <!-- <origin xyz="0 -0.09677 0" rpy="${pi/2} 0 ${pi}"/> -->
             <geometry>
                 <cylinder length="${shoulder_length}" radius="${shoulder_radius}" />
-                 <!-- <mesh filename="package://3_link_arm/meshes/puma_link2.stl" scale="0.0254 0.0254 0.0254"/> -->
             </geometry>
             <material name="blue" />
@@ -106,8 +101,6 @@
         <visual>
             <origin xyz="${link_2_length/2} 0 0" rpy="0 ${pi/2} 0"/>
-            <!-- <origin xyz="0 0 0" rpy="0 0 0"/> -->
             <geometry>
                 <cylinder length="${link_2_length}" radius="${link_2_radius}" />
-                 <!-- <mesh filename="package://3_link_arm/meshes/puma_link3.stl" scale="0.0254 0.0254 0.0254"/> -->
             </geometry>
             <material name="orange" />
@@ -138,8 +131,6 @@
         <visual>
             <origin xyz="0 -${link_3_length/2} 0" rpy="${-pi/2} 0 0"/>
-            <!-- <origin xyz="0 ${0.094/2} 0" rpy="0 0 ${-pi/2}"/> -->
             <geometry>
                 <cylinder length="${link_3_length}" radius="${link_3_radius}" />
-                 <!-- <mesh filename="package://3_link_arm/meshes/puma_link4.stl" scale="0.0254 0.0254 0.0254"/> -->
             </geometry>
             <material name="yellow" />
